File: laser_nephelometer/laser_nephelometer.kicad_sch (KiCad schematic)
At the start: 0 parts

Commit message: Checking in
Parts:
- added C1, C10, C11, C12, C13, C14, C15, C16, C17, C18, C19, C2, C24, C6, C7, C8, C9: 0.1uF, PCM_SparkFun-Capacitor:C_0402_1005Metric, symbol PCM_SparkFun-Capacitor:0.1uF_0402_16V_10%
- added C20, C21, C22, C23: 4.7uF, PCM_SparkFun-Capacitor:C_0402_1005Metric, symbol PCM_SparkFun-Capacitor:4.7uF_0402_6.3V_10%
- added C25, C26: 15pF, PCM_SparkFun-Capacitor:C_0402_1005Metric, symbol PCM_SparkFun-Capacitor:15pF_0402_50V_5%
- added C3, C4, C5: 10uF, PCM_SparkFun-Capacitor:C_0402_1005Metric, symbol PCM_SparkFun-Capacitor:10uF_0402_6.3V_20%
- added D2: Red, PCM_SparkFun-LED:LED_0402_1005Metric_Red, symbol PCM_SparkFun-LED:LED_Red_0402
- added FB1: 600 @ 100MHz, Inductor_SMD:L_0603_1608Metric, symbol Device:FerriteBead
- added J1: TYPE-C-31-M-12, TYPE-C-31-M-12:HRO_TYPE-C-31-M-12, symbol TYPE-C-31-M-12:TYPE-C-31-M-12
- added J2: SM03B-SRSS-TB_LF__SN_, SM03B-SRSS-TB_LF__SN_:JST_SM03B-SRSS-TB_LF__SN_, symbol SM03B-SRSS-TB_LF__SN_:SM03B-SRSS-TB_LF__SN_
- added L1: 2.2nH, PCM_SparkFun-Capacitor:C_0402_1005Metric, symbol PCM_SparkFun-Coil:47nH_0402_0.3A
- added L2: AOTA-B201610S3R3-101-T, AOTAB201610S3R3101T:AOTAB201610S3R3101T, symbol AOTA-B201610S3R3-101-T:AOTA-B201610S3R3-101-T
- added R1, R2: 5.1k, PCM_SparkFun-Resistor:R_0402_1005Metric, symbol PCM_SparkFun-Resistor:5.1k_0402
- added R27: 100, PCM_SparkFun-Resistor:R_0402_1005Metric, symbol PCM_SparkFun-Resistor:100_0402
- added R3: 33, PCM_SparkFun-Resistor:R_0402_1005Metric, symbol PCM_SparkFun-Resistor:33_0402
- added R4, R5, R7: 1k, PCM_SparkFun-Resistor:R_0402_1005Metric, symbol PCM_SparkFun-Resistor:1k_0402
- added R6: 10k, PCM_SparkFun-Resistor:R_0402_1005Metric, symbol PCM_SparkFun-Resistor:10k_0402
- added SW1, SW2: KMR221GLFS, PCM_SparkFun-Switch:Push_SMD_4.6x2.8mm_h1.9mm, symbol PCM_SparkFun-Switch:SPST_Push_SMD_4.6x2.8mm_h1.9mm
- added U1: USBLC6-2SC6, Package_TO_SOT_SMD:SOT-23-6, symbol Power_Protection:USBLC6-2SC6
- added U2: AP2112K-3.3, PCM_SparkFun-Semiconductor-Standard:SOT23-5, symbol PCM_SparkFun-Regulator:AP2112K-3.3
- added U3: RP2354B, Package_DFN_QFN:QFN-80-1EP_10x10mm_P0.4mm_EP3.4x3.4mm, symbol MCU_RaspberryPi:RP2354B
- added U4: APS6404L-3SQR-ZR, APS6404L-3SQR-ZR:PSON50P200X300X50-9N, symbol APS6404L-3SQR-ZR:APS6404L-3SQR-ZR
- added Y1: ABM8-272-T3, ABM8-272-T3:XTAL_ABM8-272-T3, symbol ABM8-272-T3:ABM8-272-T3
Connections:
- new net: C22.1, R3.1, U3.61 (VREG_AVDD)
- new net: J1.B5 (CC2), R1.2
- new net: J1.A5 (CC1), R2.2
- new net: L2.1, U3.63 (VREG_LX)
- new net: C26.1, R7.1, Y1.3
- new net 1.1V: C18.1, C19.1, C20.1, C23.1, L2.2, U3.10 (DVDD), U3.32 (DVDD), U3.51 (DVDD), U3.65 (VREG_FB)
- new net 3.3V: C10.1, C11.1, C12.1, C13.1, C14.1, C15.1, C16.1, C17.1, C21.1, C24.1, C4.1, C7.1, C8.1, C9.1, FB1.1, R3.2, R6.2, U2.5 (VOUT), U3.15 (IOVDD), U3.24 (IOVDD), U3.29 (IOVDD), U3.41 (IOVDD), U3.5 (IOVDD), U3.50 (IOVDD), U3.59 (ADC_AVDD), U3.60 (IOVDD), U3.64 (VREG_VIN), U3.68 (USB_OTP_VDD), U3.69 (QSPI_IOVDD), U3.76 (IOVDD), U4.8 (VDD)
- new net 5V: C2.1, C3.1, L1.2, U1.5 (VBUS), U2.1 (VIN), U2.3 (EN)
- new net ADS115_ALRT: U3.20 (GPIO20)
- new net GND: C1.2, C10.2, C11.2, C12.2, C13.2, C14.2, C15.2, C16.2, C17.2, C18.2, C19.2, C2.2, C20.2, C21.2, C22.2, C23.2, C24.2, C25.2, C26.2, C3.2, C4.2, C5.2, C6.2, C7.2, C8.2, C9.2, D2.1 (K), J1.A1_B12 (GND), J1.B1_A12 (GND__1), J1.S1 (SHIELD), J1.S2 (SHIELD__1), J1.S3 (SHIELD__2), J1.S4 (SHIELD__3), J2.2, J2.S1 (SHIELD), J2.S2 (SHIELD__1), R1.1, R2.1, R4.1, SW2.1, U1.2 (GND), U2.2 (GND), U3.62 (VREG_PGND), U3.81 (GND), U4.4 (VSS), U4.9 (EXP), Y1.2 (GND), Y1.4 (GND__1)
- new net GPIO8_(UART1_TX): U3.6 (GPIO8)
- new net GPIO9_(UART1_RX): U3.7 (GPIO9)
- new net I2C_SCL: U3.2 (GPIO5)
- new net I2C_SDA: U3.1 (GPIO4)
- new net LED: D2.2 (A), R27.2
- new net LED.R: R27.1, U3.11 (GPIO12)
- new net NEOPIXEL_IN: U3.27 (GPIO26)
- new net PICO (GPIO24): U3.25 (GPIO24)
- new net PWM_LASER: U3.22 (GPIO22)
- new net QSPI_SCLK: U3.71 (QSPI_SCLK), U4.6 (SCLK)
- new net QSPI_SD0: U3.72 (QSPI_SD0), U4.5 (SI/SIO(0))
- new net QSPI_SD1: U3.74 (QSPI_SD1), U4.2 (SO/SIO(1))
- new net QSPI_SD2: U3.73 (QSPI_SD2), U4.3 (SIO(2))
- new net QSPI_SD3: U3.70 (QSPI_SD3), U4.7 (SIO(3))
- new net RES.BUTTON: R4.2, SW1.1
- new net RTC_INT: U3.21 (GPIO21)
- new net SCLK(GPIO29): U3.37 (GPIO29)
- new net SPI_MISO: U3.16 (GPIO16)
- new net SPI_MOSI: U3.19 (GPIO19)
- new net SPI_SCK: U3.18 (GPIO18)
- new net SWCLK: J2.1, U3.33 (SWCLK)
- new net SWDIO: J2.3, U3.34 (SWDIO)
- new net USBC.D+: J1.A6 (DP1), J1.B6 (DP2), U1.3 (I/O2)
- new net USBC.D-: J1.A7 (DN1), J1.B7 (DN2), U1.1 (I/O1)
- new net USBLC6.D+: U1.4 (I/O2), U3.67 (USB_DP)
- new net USBLC6.D-: U1.6 (I/O1), U3.66 (USB_DM)
- new net VDDA: C5.1, C6.1, FB1.2
- new net VUSB: C1.1, J1.A4_B9 (VBUS), J1.B4_A9 (VBUS__1), L1.1
- new net V_TRANS: U3.49 (GPIO40/ADC0)
- new net WIFI_BLE_ON(GPIO23): U3.23 (GPIO23)
- new net XIN: C25.1, U3.30 (XIN), Y1.1
- new net XOUT: R7.2, U3.31 (XOUT)
- new net ~{BOOT}: R5.1, SW2.2
- new net ~{CS(GPIO25)}: U3.26 (GPIO25)
- new net ~{MEM_CS}: U3.17 (GPIO17)
- new net ~{PSRAM_CS}: R6.1, U3.77 (GPIO0), U4.1 (~{CE})
- new net ~{QSPI_SS}: R5.2, U3.75 (~{QSPI_SS})
- new net ~{RESET}: SW1.2, U3.35 (RUN)
- no-connect marks 0 -> 31
Other:
- removed sheet Power_Supply
- added sheet Analog_Sheet (analog_sheet.kicad_sch)
- added sheet Peripherals Sheet (Peripherals.kicad_sch)
